File: LiPo_GNSS_debug.kicad_sch (KiCad schematic)
At the start: 8 parts

Commit message: lipo_gnss_debug
Parts:
- removed R1: R_Small, symbol Device:R_Small
- added C?: 10uF, symbol Device:C_Small
- added C?: 100nF, symbol Device:C_Small
- added C?: C_Feedthrough, symbol Device:C_Feedthrough
- added C?: 1uF, symbol Device:C_Small
- added J?: Conn_01x02, Connector_JST:JST_XH_B1B-XH-AM_1x01_P2.50mm_Vertical, symbol Connector_Generic:Conn_01x02
- added J?: Conn_Coaxial, symbol Connector:Conn_Coaxial
- added L?: 27nH, symbol Device:L_Small
- added R? (x2): 10k, symbol Device:R_Small
- added R?: 10, symbol Device:R_Small
- added U1: NEO-M8N, RF_GPS:ublox_NEO, symbol RF_GPS:NEO-M8N
Connections:
- net +3.3V: now also J?.2 (Pin_2), J?.MP (MountPin), R?.1, U?.10 (GND), U?.11 (RF_IN), U?.12 (GND), U?.13 (GND), U?.2 (V_{SS}), U?.22 (V_BCKP), U?.24 (GND), U?.7 (VDD_USB), C?.1, C?.1, C?.1, C?.2, C?.2, C?.2, C?.2, J?.1 (In), J?.1 (Pin_1), J?.2 (Ext), L?.2, R?.2, R?.2, U1.10 (GND), U1.12 (GND), U1.13 (GND), U1.23 (VCC), U1.24 (GND)
- net RX2: now also U1.20 (TXD/SPI_MISO)
- net TX2: now also U1.21 (RXD/SPI_MOSI)
- net TP: now reaches U?.3 (TIMEPULSE)
- net at U?.8 (~{RESET}): now also R?.1
- net at U?.9 (VCC_RF): now also R?.1
- removed net GND: J?.2 (Pin_2), J?.MP (MountPin), R?.1, U?.10 (GND), U?.12 (GND), U?.13 (GND), U?.2 (D_SEL), U?.2 (V_{SS}), U?.24 (GND)
- new net: C?.1, R?.2
- new net: C?.3, L?.1
- new net: J?.2 (Pin_2), R?.1, U?.2 (D_SEL)
- no-connect marks 0 -> 3
Other:
- note added: "If only Uart"
- moved on the sheet: U?

Commit message: gnss_lipo_debug_temp
Parts:
- added C1: 100nF, symbol Device:C_Small
- added C2: 1uF, symbol Device:C_Small
- added C3: 10uF, symbol Device:C_Small
- added C4: C_Feedthrough, symbol Device:C_Feedthrough
- added C5, C?: 4.7uF, symbol Device:C_Small
- added C6: 0.1uF, symbol Device:C_Small
- added J2: Conn_Coaxial, symbol Connector:Conn_Coaxial
- added L1: 27nH, symbol Device:L_Small
- added R3: 10, symbol Device:R_Small
- added R? (x2): 10k, symbol Device:R_Small
- added TP1: TestPoint, symbol Connector:TestPoint
- added U?: MCP9808_MSOP, Package_SO:MSOP-8_3x3mm_P0.65mm, symbol Sensor_Temperature:MCP9808_MSOP
Connections:
- net +3.3V: now also U1.11 (RF_IN), U1.22 (V_BCKP), U1.7 (VDD_USB), C1.2, C2.1, C2.2, C3.1, C3.2, C4.2, C5.1, C6.1, C6.2, C?.1, J2.1 (In), J2.2 (Ext), L1.2, R?.1, R?.1, U?.4 (GND), U?.5 (A2), U?.6 (A1), U?.7 (A0), U?.8 (V_{DD})
- net TP: now also U1.3 (TIMEPULSE)
- net VBUS: now also C5.2
- net at U1.9 (VCC_RF): now also R3.1
- net LiPo_4.2V renamed V_BAT
- net V_BAT: now also C?.2
- new net: C4.1, R3.2
- new net: C4.3, L1.1
- new net SCL: R?.2, U?.2 (SCL)
- new net SDA: R?.2, U?.1 (SDA)
- no-connect marks 3 -> 0
Other:
- note added: "Controlled impedence of 50ohm to connect RF_IN to antenna/connector"
- moved on the sheet: C?, D?, J?, L?, R?, U?

Commit message: lipo_gnss_debug
Parts:
- added U2: MCP73833-xxx-UN, Package_SO:MSOP-10_3x3mm_P0.5mm, symbol Battery_Management:MCP73833-xxx-UN
Connections:
- new net: U2.1 (V_{DD}), U2.2 (V_{DD})
- new net: U2.10 (V_{BAT}), U2.9 (V_{BAT})
Changed lines of the file:
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@@
+	)
+	(symbol
+		(lib_id "Battery_Management:MCP73833-xxx-UN")
+		(at 40.64 93.98 0)
+		(unit 1)
+		(exclude_from_sim no)
+		(in_bom yes)
+		(on_board yes)
+		(dnp no)
+		(fields_autoplaced yes)
+		(property "Reference" "U2"
+			(at 40.64 81.28 0)
+			(effects
+				(font
+					(size 1.27 1.27)
+				)
+			)
+		)
+		(property "Value" "MCP73833-xxx-UN"
+			(at 40.64 83.82 0)
+			(effects
+				(font
+					(size 1.27 1.27)
+				)
+			)
+		)
+		(property "Footprint" "Package_SO:MSOP-10_3x3mm_P0.5mm"
+			(at 60.96 102.87 0)
+			(effects
+				(font
+					(size 1.27 1.27)
+				)
+				(hide yes)
+			)
+		)
+		(property "Datasheet" "https://ww1.microchip.com/downloads/aemDocuments/documents/OTH/ProductDocuments/DataSheets/22005b.pdf"
+			(at 40.64 93.98 0)
+			(effects
+				(font
+					(size 1.27 1.27)
+				)
+				(hide yes)
+			)
+		)
+		(property "Description" "Stand-Alone Linear Li-Ion / Li-Polymer Charge Management Controller, MSOP-10"
+			(at 40.64 93.98 0)
+			(effects
+				(font
+					(size 1.27 1.27)
+				)
+				(hide yes)
+			)
+		)
+		(pin "3"
+		)
+		(pin "6"
+		)
+		(pin "10"
+		)
+		(pin "5"
+		)
+		(pin "1"
+		)
+		(pin "2"
+		)
+		(pin "8"
+		)
+		(pin "9"
+		)
+		(pin "4"
+		)
+		(pin "7"
+		)
+		(instances
+			(project ""
+				(path "/9841acd6-84c9-43b3-bb27-06c48da1b9d4"
+					(reference "U2")
+					(unit 1)
+				)
+			)
+		)
 	)
 	(symbol

Commit message: draft
Parts:
- removed J?: SM03B-SRSS-TB, Connector_JST:JST_SH_SM03B-SRSS-TB_1x03-1MP_P1.00mm_Horizontal, symbol Connector_Generic_MountingPin:Conn_01x03_MountingPin
- removed R?: 22, symbol Device:R_Small
- removed U2: MCP73833-xxx-UN, Package_SO:MSOP-10_3x3mm_P0.5mm, symbol Battery_Management:MCP73833-xxx-UN
Other:
- note removed: "JST Debug Connector"

Commit message: draft
Parts:
- added C10: C_Feedthrough, symbol Device:C_Feedthrough
- added C7: 100nF, symbol Device:C_Small
- added C8: 1uF, symbol Device:C_Small
- added C9: 10uF, symbol Device:C_Small
- added J1: Conn_01x02, Connector_JST:JST_XH_B1B-XH-AM_1x01_P2.50mm_Vertical, symbol Connector_Generic:Conn_01x02
- added J3: Conn_Coaxial, symbol Connector:Conn_Coaxial
- added L2: 27nH, symbol Device:L_Small
- added R1: 10, symbol Device:R_Small
- added R1, R2: 10k, symbol Device:R_Small
- added U2: NEO-M8N, RF_GPS:ublox_NEO, symbol RF_GPS:NEO-M8N
Connections:
- net +3.3V: now also C10.2, C7.1, C7.2, C8.1, C8.2, C9.1, C9.2, J1.1 (Pin_1), J3.1 (In), J3.2 (Ext), L2.2, R1.2, R2.2, U2.10 (GND), U2.11 (RF_IN), U2.12 (GND), U2.13 (GND), U2.22 (V_BCKP), U2.23 (VCC), U2.24 (GND), U2.7 (VDD_USB)
- net RX2: now also U2.20 (TXD/SPI_MISO)
- net TP: now also U2.3 (TIMEPULSE)
- net TX2: now also U2.21 (RXD/SPI_MOSI)
- new net: R1.1, U2.9 (VCC_RF)
- new net: C10.1, R1.2
- new net: J1.2 (Pin_2), R1.1, U2.2 (D_SEL)
- new net: C10.3, L2.1
- new net: R2.1, U2.8 (~{RESET})
