File: Power.kicad_sch (KiCad schematic)
At the start: 0 parts

Commit message: Power
Parts:
- added C5, C?: 4.7uF, symbol Device:C_Small
- added D?: LED, symbol Device:LED
- added R?: 1k, symbol Device:R_Small
- added R?: 2k, symbol Device:R_Small
- added U1: MCP73812T-420I-OT, Package_TO_SOT_SMD:SOT-23-5, symbol Battery_Management:MCP73812T-420I-OT
- added U?: MCP73831-2-OT, Package_TO_SOT_SMD:SOT-23-5, symbol Battery_Management:MCP73831-2-OT
Connections:
- new net: R?.1, U?.1 (STAT)
- new net: D?.1 (K), R?.2
- new net: R?.2, U?.5 (PROG)
- new net GND: C5.1, C?.1, R?.1, U?.2 (V_{SS})
- new net VBUS: C5.2, D?.2 (A), U?.4 (V_{DD})
- new net V_BAT: C?.2, U?.3 (V_{BAT})
Other:
- note added: "LiPo Charger"

Commit message: Power
Parts:
- removed U1: MCP73812T-420I-OT, Package_TO_SOT_SMD:SOT-23-5, symbol Battery_Management:MCP73812T-420I-OT
- added Q1: IRLML6401, Package_TO_SOT_SMD:SOT-23, symbol Transistor_FET:IRLML6401
- added R3: 10k, symbol Device:R_Small
Connections:
- net GND: now also R3.2
- net V_BAT: now also Q1.2 (S)
- new net: Q1.1 (G), R3.1
- new net +3.3V: Q1.3 (D)
