File: Power.kicad_sch (KiCad schematic)
At the start: 0 parts

Commit message: Add files via upload
Parts:
- added BT1: 18650 LiPo, parallel18650:18650-PC4, symbol Device:Battery_Cell
- added C17, C18: 10u, Capacitor_SMD:C_0603_1608Metric, symbol Device:C
- added C19, C20: 10u, Capacitor_SMD:C_0402_1005Metric, symbol Device:C
- added C21, C23, C24, C25: 22u, Capacitor_SMD:C_0805_2012Metric, symbol Device:C
- added C22: 10u, Capacitor_SMD:C_0805_2012Metric, symbol Device:C
- added D4: YELLOW, LED_SMD:LED_0805_2012Metric, symbol Device:LED
- added D5: SS36-E3/57T, Diode_SMD:D_SMC, symbol Diode:MBRS340
- added D6: YELLOW, LED_SMD:LED_0603_1608Metric, symbol Device:LED
- added D7: GREEN, LED_SMD:LED_0603_1608Metric, symbol Device:LED
- added J6: USB_C_USB2.0_16P, Connector_USB:USB_C_Receptacle_Molex_105450-0101, symbol Connector:USB_C_Receptacle_USB2.0_16P
- added L2: 1u, easyeda2kicad:IND-SMD_L4.0-W4.0_XFL4020-102MEB, symbol Device:L
- added Q1: Si2301CDS, Package_TO_SOT_SMD:SOT-23, symbol Transistor_FET:DMG2301L
- added R15, R16: 5k1, Resistor_SMD:R_0402_1005Metric, symbol Device:R
- added R17: 5K1, Resistor_SMD:R_0402_1005Metric, symbol Device:R
- added R18: 2k2, Resistor_SMD:R_0402_1005Metric, symbol Device:R
- added R19: 10k, Resistor_SMD:R_0603_1608Metric, symbol Device:R
- added R20: 200k, Resistor_SMD:R_0402_1005Metric, symbol Device:R
- added R21: 49k9, Resistor_SMD:R_0402_1005Metric, symbol Device:R
- added R22, R23: 2k2, Resistor_SMD:R_0603_1608Metric, symbol Device:R
- added SW3: CHRG_EN, symbol Switch:SW_SPDT
- added U3: TP4056, Package_SO:SOIC-8-1EP_3.9x4.9mm_P1.27mm_EP2.41x3.3mm_ThermalVias, symbol Battery_Management:TP4056-42-ESOP8
- added U4: AMS1117-3.3, Package_TO_SOT_SMD:SOT-223-3_TabPin2, symbol Regulator_Linear:AMS1117-3.3
- added U5: TPS61230DRCR, Package_SON:Texas_S-PVSON-N10_ThermalVias, symbol Regulator_Switching:TPS61230DRC
Connections:
- new net: C19.1, C21.1, D5.1 (K), L2.1, Q1.2 (S), U4.3 (VI), U5.10 (VIN), U5.9 (EN)
- new net: R20.2, R21.1, U5.7 (FB)
- new net: L2.2, U5.1 (SW), U5.2 (SW)
- new net: C22.1, U5.6 (SS)
- new net +3V3: C20.1, D6.2 (A), U4.2 (VO)
- new net +5V: C23.1, C24.1, C25.1, D7.2 (A), R20.1, U5.3 (VOUT), U5.4 (VOUT)
- new net +BATT: BT1.1 (+), C18.1, Q1.3 (D), U3.5 (BAT)
- new net CE: SW3.2 (B), U3.8 (CE)
- new net CHRG_LED: D4.1 (K), R17.1
- new net GND: BT1.2 (-), C17.2, C18.2, C19.2, C20.2, C21.2, C22.2, C23.2, C24.2, C25.2, J6.A1 (GND), J6.A12 (GND), J6.B1 (GND), J6.B12 (GND), R15.2, R16.2, R18.2, R19.2, R21.2, R22.1, R23.1, SW3.3 (C), U3.1 (TEMP), U3.3 (GND), U3.6 (~{STDBY}), U4.1 (GND), U5.11 (GND)
- new net LED_3V3: D6.1 (K), R22.2
- new net LED_5V: D7.1 (K), R23.2
- new net PROG: R18.1, U3.2 (PROG)
- new net USB1_CC1: J6.A5 (CC1), R16.1
- new net USB1_CC2: J6.B5 (CC2), R15.1
- new net USB_D+: J6.A6 (D+), J6.B6 (D+)
- new net USB_D-: J6.A7 (D-), J6.B7 (D-)
- new net VBUS: C17.1, D4.2 (A), D5.2 (A), J6.A4 (VBUS), J6.A9 (VBUS), J6.B4 (VBUS), J6.B9 (VBUS), Q1.1 (G), R19.1, SW3.1 (A), U3.4 (V_{CC})
- new net ~{CHRG}: R17.2, U3.7 (~{CHRG})
- no-connect marks 0 -> 5
Other:
- note added: "18650 LiPo"
- note added: "Batt Charger @ 500mA"
- note added: "CHRG_EN Switch ON to charge when USB plugged in"
- note added: "Gate pulldown Avoid floating gate"
- note added: "Leave shield floating"
- note added: "Line Switcher"
- note added: "Linear +3V3 @ 1A"
- note added: "Model SYSTEM SW like "remove before flight" pin"
- note added: "Refer to Microchip AN1149"
- note added: "Rprog = 1100/Ibat 5k1 - 0.216A 2k2 - 0.5A"
- note added: "SMPS +5V @ 2A"
- note added: "Schottky Rectifier 0.45V Forward drop @ 1A, 25C 0.55V Forward drop @ 3A, 25C Tjunction higher = decrease VF"
- note added: "TVS anywhere?"
- note added: "USB-C"
- note added: "USB-C Negotiation CC1/CC2 Pull-down 5V @ 1A (nominal) 5V @ 3A (with USB-PD)"
- note added: "Vin: ~4.5V (USB) 3.0-4.2V (VBATT)"
- company: (none) -> Bronco STAR - BLV
- title: (none) -> +5V, +3V3, LiPo Battery, Charger
