File: MCU.kicad_sch (KiCad schematic)
At the start: 38 parts, among them J1 Micro_SD_Card

Commit message: Add files via upload
Parts:
- removed C?: 10u, symbol Device:C
- removed C?: 100n, symbol Device:C
- removed C?: 22u, symbol Device:C
- removed J1: Micro_SD_Card, Connector_Card:microSD_HC_Wuerth_693072010801, symbol Connector:Micro_SD_Card
- removed J?: USB_C_Receptacle_USB2.0_16P, symbol Connector:USB_C_Receptacle_USB2.0_16P
- removed L?: 3.3u, RP2350_80QFN_minimal:L_pol_2016, symbol Device:L
- removed R? (x2): 27, symbol Device:R
- removed R? (x2): 5k1, symbol Device:R
- removed U?: AMS1117-3.3, Package_TO_SOT_SMD:SOT-223-3_TabPin2, symbol Regulator_Linear:AMS1117-3.3
- added C6: 100n, Capacitor_SMD:C_0402_1005Metric, symbol Device:C
- added D1, D2, D3: GREEN, LED_SMD:LED_0805_2012Metric, symbol Device:LED
- added J5: Dupont Debug Headers, Connector_JST:JST_EH_S3B-EH_1x03_P2.50mm_Horizontal, symbol Connector:Conn_01x03_Socket
- added L1: 3.3u, RP2350_60QFN_minimal:L_pol_2016, symbol Device:L
- added R12, R13, R14: 1k, Resistor_SMD:R_0805_2012Metric, symbol Device:R
- added R2, R3: 27, Resistor_SMD:R_0402_1005Metric, symbol Device:R
- added R8, R9: 10k, Resistor_SMD:R_0402_1005Metric, symbol Device:R
- C1, C10, C11, C12, C13, C15, C16, C3, C4, C5, C7, C8, C9: renamed from C?; footprint (none) -> Capacitor_SMD:C_0402_1005Metric
- C2: renamed from C?; footprint (none) -> Capacitor_SMD:C_0603_1608Metric
- R1, R11: renamed from R?; footprint (none) -> Resistor_SMD:R_0402_1005Metric
- R10: renamed from R?; value 1k -> 10k; footprint (none) -> Resistor_SMD:R_0402_1005Metric
- R6: renamed from R?; footprint (none) -> Resistor_SMD:R_0603_1608Metric
- SW1, SW2: renamed from SW?; footprint (none) -> Button_Switch_SMD:SW_SPST_B3U-1000P
- U1: renamed from U?; footprint Package_SO:SOIC-8_5.23x5.23mm_P1.27mm -> Package_SO:SOIC-8_5.3x5.3mm_P1.27mm
- U2: renamed from U?; footprint RP2350_60QFN_minimal:RP2350-QFN-60-1EP_7x7_P0.4mm_EP3.4x3.4mm_ThermalVias -> Package_DFN_QFN:QFN-60-1EP_7x7mm_P0.4mm_EP3.4x3.4mm_ThermalVias
- gave numbers to parts that had none: 5
Connections:
- net +1V1: now also L1.1
- net +3V3: now also SW2.2, U2.26 (RUN), C6.1, R8.2, R9.2
- net GND: now also C6.2, D1.1 (K), D2.1 (K), D3.1 (K), J5.3 (Pin_3)
- net SWCLK: now also J5.1 (Pin_1)
- net SWD: now also J5.2 (Pin_2)
- net USB_D+: now also R2.1
- net USB_D-: now also R3.1
- net VREG_LX: now also L1.2
- net XOUT_R: now reaches C16.2, R11.1, Y1.3
- net BUS_SPI1_MISO: now reaches U2.16 (GPIO12)
- net BUS_SPI1_CS: now reaches U2.17 (GPIO13)
- net BUS_SPI1_SCK: now reaches U2.18 (GPIO14)
- net BUS_SPI1_MOSI: now reaches U2.19 (GPIO15)
- net RF_SPI_CS: now reaches U2.28 (GPIO17)
- net RF_SPI_SCK: now reaches U2.29 (GPIO18)
- net RF_SPI_MOSI: now reaches U2.31 (GPIO19)
- net RF_SPI_MISO: now reaches U2.32 (GPIO20)
- net BUS_I2C0_SDA: now reaches U2.36 (GPIO24)
- net BUS_I2C0_SDA: now also R8.1
- net BUS_I2C0_SCL: now reaches U2.37 (GPIO25)
- net BUS_I2C0_SCL: now also R9.1
- net at U2.4 (GPIO2): now also R12.1
- net at U2.51 (USB_DM): now also R3.2
- net at U2.52 (USB_DP): now also R2.2
- net at U2.9 (GPIO6): now also R13.1
- net CS1 renamed CUBE_UART2_RX
- net GPIO0: no longer names the net of R5.1
- net MISO1 renamed CUBE_UART2_TX
- net MOSI1: no longer names the net of U2.15 (GPIO11)
- net RX0 renamed CUBE_UART0_RX
- net RX1 renamed CUBE_UART1_RX
- net SCK1: no longer names the net of U2.14 (GPIO10)
- net SCK1: now also R14.1
- net TX0 renamed CUBE_UART0_TX
- net TX1 renamed CUBE_UART1_TX
- new net: D2.2 (A), R13.2
- new net: D3.2 (A), R14.2
- new net: D1.2 (A), R12.2
- no-connect marks 4 -> 12
Other:
- note added: "Get line characteristic impedance to 90 ohms"
- note added: "Make sure PCB trace is short"
- note added: "R < 1k for high brightness on sunny field day"
- note added: "UART TX Indicator LEDs"
- note added: "Use PIO mode as virtual UART in Software"
- note removed: "- Why are we using two separate SPI and I2C lines?"
- note removed: "SD Card (SPI Mode)"
- company: (none) -> Bronco STAR - BLV
- title: (none) -> Microcontroller RP2350A
- moved on the sheet: C14, R10, R4, R5, R7, SW2, U1
