File: Sensors.kicad_sch (KiCad schematic)
At the start: 0 parts

Commit message: sensors
Parts:
- added C6: 0.1uF, symbol Device:C_Small
- added R1, R2: 10k, symbol Device:R_Small
- added U1: MCP9808_MSOP, Package_SO:MSOP-8_3x3mm_P0.65mm, symbol Sensor_Temperature:MCP9808_MSOP
Connections:
- new net +3.3V: C6.2, R1.1, R2.1, U1.8 (V_{DD})
- new net GND: C6.1, U1.4 (GND), U1.5 (A2), U1.6 (A1), U1.7 (A0)
- new net SCL: R1.2, U1.2 (SCL)
- new net SDA: R2.2, U1.1 (SDA)
Other:
- note added: "Battery Temp Sensor"

Commit message: Sensors
Parts:
- added C1 (x2): 100nF, symbol Device:C_Small
- added C2 (x2): 1uF, symbol Device:C_Small
- added C3 (x2): 10uF, symbol Device:C_Small
- added C4 (x2): C_Feedthrough, symbol Device:C_Feedthrough
- added J2, J?: Conn_Coaxial, symbol Connector:Conn_Coaxial
- added J?: Conn_01x02, Connector_JST:JST_XH_B1B-XH-AM_1x01_P2.50mm_Vertical, symbol Connector_Generic:Conn_01x02
- added L1, L?: 27nH, symbol Device:L_Small
- added R1, R2: 10k, symbol Device:R_Small
- added R3 (x2): 10, symbol Device:R_Small
- added U1 (x2): NEO-M8N, RF_GPS:ublox_NEO, symbol RF_GPS:NEO-M8N
- renumbered C6 to C?, R2 to R?, R1 to R?, U1 to U?
Connections:
- net GND is gone; now on net +3.3V: C?.1, U?.4 (GND), U?.5 (A2), U?.6 (A1), U?.7 (A0)
- net +3.3V: now also C1.1, C1.2, C1.2, C2.1, C2.1, C2.2, C2.2, C3.1, C3.1, C3.2, C3.2, C4.2, C4.2, J2.1 (In), J2.2 (Ext), J?.1 (In), J?.1 (Pin_1), J?.2 (Ext), L1.2, L?.2, R1.2, R2.2, U1.10 (GND), U1.10 (GND), U1.11 (RF_IN), U1.11 (RF_IN), U1.12 (GND), U1.12 (GND), U1.13 (GND), U1.13 (GND), U1.22 (V_BCKP), U1.22 (V_BCKP), U1.23 (VCC), U1.23 (VCC), U1.24 (GND), U1.24 (GND), U1.7 (VDD_USB), U1.7 (VDD_USB)
- new net: J?.2 (Pin_2), R1.1, U1.2 (D_SEL)
- new net: R3.1, U1.9 (VCC_RF) (x2)
- new net: C4.1, R3.2 (x2)
- new net: C4.3, L?.1
- new net: C4.3, L1.1
- new net: R2.1, U1.8 (~{RESET})
- new net RX2: U1.20 (TXD/SPI_MISO), U1.20 (TXD/SPI_MISO)
- new net TP: U1.3 (TIMEPULSE), U1.3 (TIMEPULSE)
- new net TX2: U1.21 (RXD/SPI_MOSI), U1.21 (RXD/SPI_MOSI)
Other:
- note added: "Controlled impedence of 50ohm to connect RF_IN to antenna/connector"
- note added: "GNSS"
- note added: "If only Uart"

Commit message: Sensors
Parts:
- removed C1: 100nF, symbol Device:C_Small
- removed C2: 1uF, symbol Device:C_Small
- removed C3: 10uF, symbol Device:C_Small
- removed C4 (x2): C_Feedthrough, symbol Device:C_Feedthrough
- removed J?: Conn_01x02, Connector_JST:JST_XH_B1B-XH-AM_1x01_P2.50mm_Vertical, symbol Connector_Generic:Conn_01x02
- removed J?: Conn_Coaxial, symbol Connector:Conn_Coaxial
- removed L?: 27nH, symbol Device:L_Small
- removed R1, R2: 10k, symbol Device:R_Small
- removed R3: 10, symbol Device:R_Small
- removed U1: NEO-M8N, RF_GPS:ublox_NEO, symbol RF_GPS:NEO-M8N
- added C5: 47 pF, symbol Device:C_Small
Connections:
- net +3.3V: now also C1.1, C5.2; no longer J2.1 (In), L1.2, U1.11 (RF_IN)
- net at R3.2: now also L1.1, C5.1
- net RX2 renamed RX
- net TP: no longer names the net of U1.3 (TIMEPULSE)
- net TX2 renamed TX
- new net: J2.1 (In), L1.2, U1.11 (RF_IN)
Other:
- note removed: "If only Uart"
- moved on the sheet: C1, C2, C3, C?, J2, L1, R3, R?, U1, U?

Commit message: sensors
Parts:
- added C4: 100nF, symbol Device:C_Small
- added C6: 1uF, symbol Device:C_Small
- added C7: 10uF, symbol Device:C_Small
- added R1: 10k, symbol Device:R_Small
- added U2: NEO-M8N, RF_GPS:ublox_NEO, symbol RF_GPS:NEO-M8N
- added U3: SKY65404, RF:Skyworks_SKY65404-31, symbol RF_Amplifier:SKY65404
Connections:
- net +3.3V: now also C4.1, C4.2, C6.1, C6.2, C7.1, C7.2, R1.1, U2.10 (GND), U2.12 (GND), U2.13 (GND), U2.2 (D_SEL), U2.22 (V_BCKP), U2.23 (VCC), U2.24 (GND), U2.7 (VDD_USB)
- new net: U3.2 (GND), U3.5 (GND)
- new net CLK: U2.19 (SCL/SPI_CLK)
- new net CS: U2.18 (SDA/~{SPI_CS})
- new net EN: R1.2, U2.14 (LNA_EN)
- new net MISO: U2.20 (TXD/SPI_MISO)
- new net MOSI: U2.21 (RXD/SPI_MOSI)
- new net RF_OUT: U2.11 (RF_IN)
- new net VCC: U2.9 (VCC_RF)

Commit message: Sensors
Parts:
- removed U3: SKY65404, RF:Skyworks_SKY65404-31, symbol RF_Amplifier:SKY65404
- added R4: 1k, symbol Device:R_Small
- added SW1: SW_Push, symbol Switch:SW_Push
Connections:
- net +3.3V: now also R4.2; no longer U2.7 (VDD_USB)
- net USB_DM: now reaches U2.5 (USB_DM)
- net USB_DP: now reaches U2.6 (USB_DP)
- net at U2.8 (~{RESET}): now also SW1.2
- net RF_OUT renamed RF_IN
- net VCC: no longer names the net of U2.9 (VCC_RF)
- new net: R4.1, SW1.1
- new net VBUS: U2.7 (VDD_USB)
- no-connect marks 0 -> 1
Other:
- note added: "(EXTINT) Wake up from power saving mode"
- note added: "(SAFEBOOT) For future service, updates and reconfiguration, leave OPEN"
- note added: "(TIMEPULSE)Configurable Timepulse 1 signal (one pulse per second by default)."

Commit message: Sensors
Parts:
- removed C3: 10uF, symbol Device:C_Small
- removed C5: 47 pF, symbol Device:C_Small
- removed C?: 0.1uF, symbol Device:C_Small
- removed J2: Conn_Coaxial, symbol Connector:Conn_Coaxial
- removed L1: 27nH, symbol Device:L_Small
- removed R3: 10, symbol Device:R_Small
- removed U1: NEO-M8N, RF_GPS:ublox_NEO, symbol RF_GPS:NEO-M8N
- added J1: USB_B_Micro, symbol Connector:USB_B_Micro
- added R10, R11, R9: 10k, symbol Device:R_Small
- added R12: 100k, symbol Device:R_Small
- added R13: 2k, symbol Device:R_Small
- added R2, R5: 27, symbol Device:R_Small
- added R6: 1k, symbol Device:R_Small
- added R8: 4.7k, symbol Device:R_Small
- added U1: AMS1117-3.3, Package_TO_SOT_SMD:SOT-223-3_TabPin2, symbol Regulator_Linear:AMS1117-3.3
- C1: value 100nF -> 22uF
- C2: value 1uF -> 10uF
Connections:
- net USB_DM: now also J1.2 (D-), R2.2; no longer U2.5 (USB_DM)
- net USB_DP: now also J1.3 (D+), R5.2; no longer U2.6 (USB_DP)
- net Alert: now reaches U?.3 (Alert)
- net Alert: now also R8.2
- net +3.3V renamed +3V3
- net +3V3: now also J1.5 (GND), J1.6 (Shield), R10.2, R11.2, R12.1, R13.1, R13.2, R6.2, R8.1, R9.2, U1.1 (GND), U1.2 (VO); no longer C2.2, U?.5 (A2), U?.6 (A1), U?.7 (A0)
- net VBUS: no longer names the net of U2.7 (VDD_USB)
- net VBUS: now also R12.2
- new net: R2.1, U2.5 (USB_DM)
- new net: R5.1, U2.6 (USB_DP)
- new net: R11.1, U?.5 (A2)
- new net: R9.1, U?.6 (A1)
- new net: R10.1, U?.7 (A0)
- new net VBUS2: C2.2, J1.1 (VBUS), U1.3 (VI)
- no-connect marks 1 -> 2
Other:
- note removed: "Controlled impedence of 50ohm to connect RF_IN to antenna/connector"
- moved on the sheet: C4, C6, C7, R1, R4, R?, SW1, U2
