File: Sensors.kicad_sch (KiCad schematic)
At the start: 0 parts

Commit message: Add files via upload
Other:
- note added: "Temp Sensor?"
- company: (none) -> Bronco STAR - BLV
Changed lines of the file:
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@@
 	(generator "eeschema")
 	(generator_version "9.0")
-	(paper "A4")
+	(paper "USLedger")
+	(title_block
+		(date "2025-07-01")
+		(rev "A")
+		(company "Bronco STAR - BLV")
+	)
+	(text "Temp Sensor?"
+		(exclude_from_sim no)
+		(at 53.594 36.83 0)
+		(effects
+			(font
+				(size 2.54 2.54)
+				(thickness 0.508)
+				(bold yes)
+			)
+		)
+	)
 )
