File: BLV_PCB.kicad_sch (KiCad schematic)
At the start: 0 parts

Commit message: Add files via upload
Parts:
- added H1, H2, H3, H4: MountingHole, MountingHole:MountingHole_3.2mm_M3, symbol Mechanical:MountingHole
- added J1, J2, J3: Cube0 JST-PH, Connector_JST:JST_PH_S4B-PH-K_1x04_P2.00mm_Horizontal, symbol Connector:Conn_01x04_Socket
- added J4: Micro_SD_Card, Connector_Card:microSD_HC_Wuerth_693072010801, symbol Connector:Micro_SD_Card
Connections:
- new net +3V3: J4.4 (VDD)
- new net GND: J1.4 (Pin_4), J2.4 (Pin_4), J3.4 (Pin_4), J4.6 (VSS), J4.9 (SHIELD)
- new net GNSS/SPI_CS: J4.2 (DAT3/CD)
- new net GNSS/SPI_MISO: J4.7 (DAT0)
- new net GNSS/SPI_MOSI: J4.3 (CMD)
- new net GNSS/SPI_SCK: J4.5 (CLK)
- new net MCU/CUBE_UART0_RX: J1.2 (Pin_2)
- new net MCU/CUBE_UART0_TX: J1.1 (Pin_1)
- new net MCU/CUBE_UART1_RX: J2.2 (Pin_2)
- new net MCU/CUBE_UART1_TX: J2.1 (Pin_1)
- new net MCU/CUBE_UART2_RX: J3.2 (Pin_2)
- new net MCU/CUBE_UART2_TX: J3.1 (Pin_1)
- no-connect marks 0 -> 8
Other:
- added sheet GNSS (GNSS.kicad_sch)
- added sheet RF (RF.kicad_sch)
- sheet MCU ports: added BUS_I2C0_SCL, BUS_I2C0_SDA, BUS_SPI1_CS, BUS_SPI1_MISO, BUS_SPI1_MOSI, BUS_SPI1_SCK, CUBE_UART0_RX, CUBE_UART0_TX, CUBE_UART1_RX, CUBE_UART1_TX, CUBE_UART2_RX, CUBE_UART2_TX, RF_SPI_CS, RF_SPI_MISO, RF_SPI_MOSI, RF_SPI_SCK; removed none
- note added: "Check with BLV requirements matrix"
- note added: "MicroSD (SPI Mode)"
- company: (none) -> Bronco STAR - BLV
